Commit message: patrol working fine

File: tb4_openx_description/urdf/create3.urdf.xacro (robot description, xacro)
@@ -274,5 +274,5 @@
     <gazebo>
       <plugin filename="libignition-gazebo-sensors-system.so" name="ignition::gazebo::systems::Sensors">
-        <render_engine>ogre</render_engine>
+        <render_engine>ogre2</render_engine>
       </plugin>
     </gazebo>

File: tb4_openx_description/urdf/t4_manipulator.urdf.xacro (robot description, xacro)
@@ -28,5 +28,5 @@
   </gazebo>
   <xacro:arm name="arm" parent_link="$(arg prefix)link5" model="pro">
-    <origin xyz="0.070 0.0 0.052" rpy="0 0 0"/>
+    <origin xyz="0.070 0.0 0.06" rpy="0 0 0"/>
   </xacro:arm>
   <joint name="$(arg prefix)world_fixed" type="fixed">
