Commit message: added nav alignment

File: tb4_openx_description/models/artag/artag.urdf.xacro (robot description, xacro)
@@ -10,4 +10,5 @@
   <link name="artag">
     <visual>
+      <origin xyz="0 0 0" rpy="0 0 0"/>
       <geometry>
         <mesh filename="file://$(find tb4_openx_description)/models/artag/meshes/artag.dae"/>
